File: rev_a/bus_power.sch (KiCad schematic (older format))
At the start: 14 parts, among them Q1 FQP47P06, Q2 FQP47P06, SW1 F-426-0020

Commit message: Finnished Revision A layout.
Parts:
- removed N1: MS_DATA_HEADER_POWER, symbol MS_DATA_HEADER_POWER
- removed N2: MS_PWR_HEADER_POWER, symbol MS_PWR_HEADER_POWER
- added H2, H3, H4: 3MM_HOLE, symbol 3MM_HOLE
- added J1: TERMINATE_JUMPER, symbol TERMINATE_JUMPER
- added N2: BUS_MASTER_HEADER, symbol BUS_MASTER_HEADER
- added R1: 120 1%, symbol R_HORIZ
- R3: renamed from R2; value RESETABLE_FUSE -> MF-R300
- renumbered R1 to R2
Connections:
- net GND renamed LGND
- net LGND: now also H2.1 (GND), H3.1 (GND), H4.1 (GND), N2.3 (LGND1), N2.4 (LGND2)
- net MGND: no longer names the net of N4.1 (-), N5.1 (-), Q1.G
- net MGND: now also N2.7 (BGND1), N2.8 (BGND2)
- net MPWR: no longer names the net of SW1.2
- net MPWR: now also N2.10 (BPWR2), N2.9 (BPWR1)
- net VIN: no longer names the net of SW1.5
- net VIN: now also N2.1 (LPWR1), N2.2 (LPWR2)
- new net: J1.1 (ON), N2.5 (CANH)
- new net: J1.2 (COM), R1.1
- new net: N2.6 (CANL), R1.2
- no-connect marks 26 -> 3
Other:
- moved on the sheet: H1, SW1
