File: rev_b/$bus_power.sch (KiCad schematic (older format))
At the start: 18 parts, among them J1 TERMINATE_JUMPER, Q1 FQP47P06, Q2 FQP47P06, SW1 F-426-0020

Commit message: Did first layout of Rev. B.
Connections:
- net LPWR4: no longer N3.2 (+), N4.2 (+)
- net MGND: now reaches N2.7 (BGND1), N2.8 (BGND2), N4.1 (-), N5.1 (-), Q1.G
- new net MPWR0: N3.2 (+), N4.2 (+)
Changed lines of the file:
@@
 $EndComp
 Text Label 2850 1600 0    50   ~ 0
-LPWR4
+MPWR0
 $Comp
 L TERMINATE_JUMPER J1
@@
 Text Label 3500 5700 0    50   ~ 0
 LPWR4
+Text Label 3500 2500 0    50   ~ 0
+MGND
 $EndSCHEMATC
